File: main-board/main-board.kicad_pcb (KiCad board)
At the start: 2 copper layers, 93 x 45 mm, 29 parts, among them J1 AC_IN, J2 AC_OUT, J3 AC_OUT, K1 SRD-05VDC-SL-C, Q1 MMBT2222ALT1G, Q2 BTA12-600B, U1 LTV-354T, U2 Arduino-nano-BLE-33, U3 FODM3022, U4 SCD40-D-R2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

Commit message: update board v1.0
Parts:
- added REF**: MountingHole_3.2mm_M3_Pad_Via, MountingHole:MountingHole_3.2mm_M3_Pad_Via, F.Cu at (80.0, 82.0)
- added REF**: MountingHole_3.2mm_M3_Pad_Via, MountingHole:MountingHole_3.2mm_M3_Pad_Via, F.Cu at (88.5, 45.0)
- added REF**: MountingHole_3.2mm_M3_Pad_Via, MountingHole:MountingHole_3.2mm_M3_Pad_Via, F.Cu at (143.0, 70.0)
- added REF**: MountingHole_3.2mm_M3_Pad_Via, MountingHole:MountingHole_3.2mm_M3_Pad_Via, F.Cu at (143.0, 45.0)
- moved REF** 22.0 mm to (110.0, 66.0)
- moved U2 1.16 mm to (112.0, 63.2)
Routing:
- net +3V3: track 88.2 -> 84.4 mm
- net GND: track 40.4 -> 37.8 mm
- net +5V: track 58.1 -> 60.0 mm
- net /ZeroDetector: track 8.65 -> 10.2 mm
- net /SDA: track 21.9 -> 20.6 mm
- net /ControlSignal2: track 13.2 -> 12.0 mm
- net /ControlSignal1: track 18.3 -> 17.3 mm
- net /SCL: track 16.1 -> 15.1 mm
- net LINE: track 223.8 -> 223.0 mm
Other:
- board text added: "Main Board"
- board text added: "v1.0"
