File: main-board/main-board.kicad_sch (KiCad schematic)
At the start: 22 parts, among them J1 AC_IN, J2 AC_OUT, J3 AC_OUT, K1 SRD-05VDC-SL-C, Q1 MMBT2222ALT1G, Q2 BTA12-600B, U1 LTV-354T, U2 Arduino-nano-BLE-33, U3 FODM3022, U4 SCD40-D-R2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

Commit message: update main board
Parts:
- added C2, C3, C4: 10uF, Capacitor_SMD:C_0805_2012Metric, symbol Device:C_Small
- added C5: 1uF, Capacitor_SMD:C_0805_2012Metric, symbol Device:C_Small
- added R8: 4.7R, Resistor_SMD:R_0805_2012Metric, symbol Device:R_Small
- F1: footprint (none) -> Fuse:Fuseholder_Littelfuse_100_series_5x20mm
Connections:
- net +3V3: now also U4.19 (VDDH), U4.7 (VDD), C2.1, C3.1, C4.1, R8.2
- net ControlSignal1: now also U2.21
- net ControlSignal2: now also U2.20
- net GND: now also U4.20 (GND_2), U4.21 (GND_3), U4.6 (GND), U5.2 (VSS), U5.4 (N/A), U5.7 (EP), C2.2, C3.2, C4.2, C5.2
- net LINE: now also F1.2, PS1.1 (AC/L), R2.1; no longer F1.1, J1.2 (Pin_2), R1.1
- net NEUT: now also R1.1; no longer R2.1
- net SCL: now also U4.9 (SCL), U5.6 (SCL)
- net SDA: now also U4.10 (SDA), U5.3 (SDA)
- net ZeroDetector: now also U2.5
- net at U5.1 (VDD): now also U5.5 (VDDH), C5.1, R8.1
- new net: F1.1, J1.2 (Pin_2)
Other:
- moved on the sheet: F1
